File: pcb/GPC_dev_board.kicad_pcb (KiCad board)
At the start: 6 copper layers, 123.1 x 59.4 mm, 83 parts, among them J1 Conn_01x12, J10 Conn_02x06_Top_Bottom, J11 Conn_02x06_Top_Bottom, J12 Conn_01x04, J13 Conn_01x04, J16 Conn_01x06, J17 Conn_01x06, J2 Conn_01x12, J3 Conn_02x13_Odd_Even, J4 Conn_02x13_Odd_Even, J5 Screw_Terminal_01x02, J6 Screw_Terminal_01x02, J7 Screw_Terminal_01x02, J8 Screw_Terminal_01x02, J9 Screw_Terminal_01x02, Q1 C3M0120100K, Q2 IRF4905, Q3 IRF4905, Q4 IRF4905, Q5 IRF4905, U1 AMC3330, U12 TLV74318, U19 XS-GPC-01, U2 AMC3330, U7 TLV74325, U9 AD7352

Commit message: In process, Dev board topology PCB sections and floorplanning evolution.
Parts:
- removed C63, C64: 10u, Capacitor_SMD:C_1206_3216Metric
- removed C67, C68: 0.1u, Capacitor_SMD:C_0603_1608Metric
- removed J13: Conn_01x04, Connector_PinHeader_2.54mm:PinHeader_1x04_P2.54mm_Vertical
- removed J8, J9: Screw_Terminal_01x02, TerminalBlock_Phoenix:TerminalBlock_Phoenix_MKDS-1,5-2-5.08_1x02_P5.08mm_Horizontal
- removed R43: 10K, Resistor_SMD:R_0603_1608Metric
- added C26: C_Polarized, Capacitor_THT:CP_Radial_D10.0mm_P5.00mm, F.Cu at (239.3, 98.6)
- added C27: C_Polarized, Capacitor_THT:CP_Radial_D10.0mm_P5.00mm, F.Cu at (251.2, 110.7)
- added C29: C_Polarized, Capacitor_THT:CP_Radial_D10.0mm_P5.00mm, F.Cu at (264.0, 98.2)
- added C3: 0.1u, Capacitor_SMD:C_0603_1608Metric, B.Cu at (104.2, 101.4)
- added C30: 22n 1000v, Capacitor_THT:C_Rect_L13.0mm_W6.0mm_P10.00mm_FKS3_FKP3_MKS4, B.Cu at (116.2, 69.1)
- added C31: 1u, Capacitor_SMD:C_0603_1608Metric, B.Cu at (121.1, 101.3)
- added C33: 0.01u, Capacitor_SMD:C_0603_1608Metric, B.Cu at (116.5, 101.3)
- added C34: 0.1u, Capacitor_SMD:C_0603_1608Metric, B.Cu at (106.8, 101.4)
- added C35: 0.1u, Capacitor_SMD:C_0603_1608Metric, B.Cu at (109.0, 101.4)
- added C37: C_Polarized, Capacitor_THT:CP_Radial_D10.0mm_P5.00mm, F.Cu at (256.3, 98.6)
- added C38: 1u, Capacitor_SMD:C_0603_1608Metric, F.Cu at (208.6, 32.3)
- added C39: 0.01u, Capacitor_SMD:C_0603_1608Metric, F.Cu at (208.6, 34.8)
- added C40: 0.1u, Capacitor_SMD:C_0603_1608Metric, F.Cu at (208.6, 37.3)
- added C41: 0.1u, Capacitor_SMD:C_0603_1608Metric, F.Cu at (216.7, 18.0)
- added C42: 0.1u, Capacitor_SMD:C_0603_1608Metric, F.Cu at (208.6, 42.3)
- added C43: 1u, Capacitor_SMD:C_0603_1608Metric, F.Cu at (208.6, 44.8)
- added C44: 0.01u, Capacitor_SMD:C_0603_1608Metric, F.Cu at (208.6, 47.3)
- added C45: 0.1u, Capacitor_SMD:C_0603_1608Metric, F.Cu at (208.6, 49.8)
- added C46: 0.1u, Capacitor_SMD:C_0603_1608Metric, F.Cu at (212.6, 32.3)
- added C47: 0.1u, Capacitor_SMD:C_0603_1608Metric, F.Cu at (220.7, 12.9)
- added C48: 1u, Capacitor_SMD:C_0603_1608Metric, F.Cu at (212.6, 37.3)
- added C49: 0.01u, Capacitor_SMD:C_0603_1608Metric, F.Cu at (212.6, 39.8)
- added C50: 0.1u, Capacitor_SMD:C_0603_1608Metric, F.Cu at (220.7, 20.5)
- added C51: 0.1u, Capacitor_SMD:C_0603_1608Metric, F.Cu at (220.7, 23.0)
- added C54: 0.1u, Capacitor_SMD:C_0603_1608Metric, F.Cu at (212.6, 47.3)
- added C55: 0.1u, Capacitor_SMD:C_0603_1608Metric, F.Cu at (212.6, 49.8)
- added C58: 2.2n 80V, Capacitor_SMD:C_0603_1608Metric, F.Cu at (216.6, 32.3)
- added C60: 2.2n 80V, Capacitor_SMD:C_0603_1608Metric, F.Cu at (216.6, 34.8)
- added C62: 2.2n 80V, Capacitor_SMD:C_0603_1608Metric, F.Cu at (216.6, 37.3)
- added C9: C_Polarized, Capacitor_THT:CP_Radial_D10.0mm_P5.00mm, F.Cu at (256.1, 87.8)
- added D1: DC UNDER, LED_SMD:LED_0603_1608Metric, F.Cu at (188.8, 158.1)
- added D2: DC OVER, LED_SMD:LED_0603_1608Metric, F.Cu at (188.7, 153.8)
- added D3: AC UNDER, LED_SMD:LED_0603_1608Metric, F.Cu at (197.2, 158.1)
- added D4: AC OVER, LED_SMD:LED_0603_1608Metric, F.Cu at (196.8, 153.8)
- added D5: 3.3V, LED_SMD:LED_0603_1608Metric, F.Cu at (165.0, 144.9)
- added H1: ~, MountingHole:MountingHole_3mm_Pad, F.Cu at (144.9, 115.0)
- added H10: ~, MountingHole:MountingHole_3mm_Pad, F.Cu at (209.4, 124.8)
- added H11: ~, MountingHole:MountingHole_3mm_Pad, F.Cu at (276.6, 72.8)
- added H13: ~, MountingHole:MountingHole_3mm_Pad, F.Cu at (104.3, 161.7)
- added H14: ~, MountingHole:MountingHole_3mm_Pad, F.Cu at (104.5, 133.2)
- added H15: ~, MountingHole:MountingHole_3mm_Pad, F.Cu at (130.7, 160.5)
- added H16: ~, MountingHole:MountingHole_3mm_Pad, F.Cu at (130.6, 133.5)
- added H2: ~, MountingHole:MountingHole_3mm_Pad, F.Cu at (186.3, 71.2)
- added H3: ~, MountingHole:MountingHole_3mm_Pad, F.Cu at (154.8, 151.0)
- added H4: ~, MountingHole:MountingHole_3mm_Pad, F.Cu at (209.1, 73.8)
- added H5: ~, MountingHole:MountingHole_3mm_Pad, F.Cu at (145.1, 71.5)
- added H6: ~, MountingHole:MountingHole_3mm_Pad, F.Cu at (252.9, 152.3)
- added H7: ~, MountingHole:MountingHole_3mm_Pad, F.Cu at (275.7, 124.8)
- added H9: ~, MountingHole:MountingHole_3mm_Pad, F.Cu at (186.9, 113.6)
- added J14: Conn_01x04, Connector_PinHeader_2.54mm:PinHeader_1x04_P2.54mm_Horizontal, F.Cu at (120.9, 108.1)
- added J15: Vdc, TerminalBlock_Phoenix:TerminalBlock_Phoenix_MKDS-1,5-2-5.08_1x02_P5.08mm_Horizontal, F.Cu at (104.2, 150.1)
- added J18: Vac, TerminalBlock_Phoenix:TerminalBlock_Phoenix_MKDS-1,5-2-5.08_1x02_P5.08mm_Horizontal, F.Cu at (104.3, 139.5)
- added J19: LVIN, Connector_PinHeader_2.54mm:PinHeader_1x04_P2.54mm_Vertical, F.Cu at (170.2, 71.5)
- added J20: LVOUT, Connector_PinHeader_2.54mm:PinHeader_1x04_P2.54mm_Horizontal, F.Cu at (128.9, 142.6)
- added PS1: RM-3.312S, Converter_DCDC:Converter_DCDC_Murata_MEE1SxxxxSC_THT, F.Cu at (216.4, 109.2)
- added PS2: RM-3.312S, Converter_DCDC:Converter_DCDC_Murata_MEE1SxxxxSC_THT, B.Cu at (107.8, 109.3)
- added PS3: RM-3.312S, Converter_DCDC:Converter_DCDC_Murata_MEE1SxxxxSC_THT, F.Cu at (216.3, 92.6)
- added PS4: RM-3.312S, Converter_DCDC:Converter_DCDC_Murata_MEE1SxxxxSC_THT, F.Cu at (215.9, 76.1)
- added Q6: MMBT3904, Package_TO_SOT_SMD:SOT-23, F.Cu at (150.5, 114.8)
- added Q7: MMBT3904, Package_TO_SOT_SMD:SOT-23, F.Cu at (154.1, 114.8)
- added Q8: MMBT3904, Package_TO_SOT_SMD:SOT-23, F.Cu at (174.5, 115.2)
- added Q9: MMBT3904, Package_TO_SOT_SMD:SOT-23, F.Cu at (178.4, 115.2)
- added R10: 47K, Resistor_SMD:R_0603_1608Metric, F.Cu at (216.6, 39.8)
- added R11: 47K, Resistor_SMD:R_0603_1608Metric, B.Cu at (116.3, 104.9)
- added R15: 100R, Resistor_SMD:R_0603_1608Metric, B.Cu at (118.6, 104.9)
- added R16: 10R, Resistor_SMD:R_0603_1608Metric, B.Cu at (110.6, 96.9)
- added R17: 47K, Resistor_SMD:R_0603_1608Metric, B.Cu at (121.1, 104.6)
- added R18: 47K, Resistor_SMD:R_0603_1608Metric, F.Cu at (216.6, 42.3)
- added R19: 100R, Resistor_SMD:R_0603_1608Metric, F.Cu at (216.6, 44.8)
- added R20: 10R, Resistor_SMD:R_0603_1608Metric, F.Cu at (216.6, 47.3)
- added R21: 47K, Resistor_SMD:R_0603_1608Metric, F.Cu at (216.6, 49.8)
- added R22: 47K, Resistor_SMD:R_0603_1608Metric, F.Cu at (220.6, 32.3)
- added R23: 100R, Resistor_SMD:R_0603_1608Metric, F.Cu at (220.6, 34.8)
- added R24: 10R, Resistor_SMD:R_0603_1608Metric, F.Cu at (220.6, 37.3)
- added R25: 10R, Resistor_SMD:R_0603_1608Metric, F.Cu at (220.6, 39.8)
- added R26: 10R, Resistor_SMD:R_0603_1608Metric, F.Cu at (220.6, 42.3)
- added R27: 100R, Resistor_SMD:R_0603_1608Metric, F.Cu at (220.6, 44.8)
- added R28: 100R, Resistor_SMD:R_0603_1608Metric, F.Cu at (220.6, 47.3)
- added R4: 1.99M, Resistor_SMD:R_2512_6332Metric, F.Cu at (122.7, 152.5)
- added R6: 100K, Resistor_SMD:R_2512_6332Metric, F.Cu at (122.2, 140.1)
- added R9: 150R 3W, Resistor_SMD:R_2512_6332Metric, F.Cu at (111.1, 69.1)
- added RV1: GAIN_SIN, Potentiometer_THT:Potentiometer_Bourns_3299X_Horizontal, F.Cu at (177.0, 151.4)
- added RV2: GAIN_OUT, Potentiometer_THT:Potentiometer_Bourns_3299X_Horizontal, F.Cu at (211.0, 151.8)
- added RV3: GAIN_AC, Potentiometer_THT:Potentiometer_Bourns_3299X_Horizontal, F.Cu at (221.0, 151.5)
- added RV4: GAIN_DC, Potentiometer_THT:Potentiometer_Bourns_3299X_Horizontal, F.Cu at (231.7, 151.4)
- added RV5: PWM_VREF, Potentiometer_THT:Potentiometer_Bourns_3299X_Horizontal, F.Cu at (242.2, 151.3)
- added U10: ISO7320FC, Package_SO:SOIC-8_3.9x4.9mm_P1.27mm, F.Cu at (221.2, 82.0)
- added U11: TLV74325, Package_TO_SOT_SMD:SOT-23-5, F.Cu at (230.6, 90.9)
- added U13: IXDN614, Package_SO:SOIC-8_3.9x4.9mm_P1.27mm, F.Cu at (230.4, 114.0)
- added U14: MAX3485, Package_SO:SOIC-8_3.9x4.9mm_P1.27mm, F.Cu at (213.3, 98.9)
- added U15: ISO7320FC, Package_SO:SOIC-8_3.9x4.9mm_P1.27mm, F.Cu at (221.3, 98.7)
- added U16: TLV74325, Package_TO_SOT_SMD:SOT-23-5, F.Cu at (229.7, 73.7)
- added U17: IXDN614, Package_SO:SOIC-8_3.9x4.9mm_P1.27mm, F.Cu at (230.0, 82.0)
- added U18: IXDN614, Package_SO:SOIC-8_3.9x4.9mm_P1.27mm, F.Cu at (230.0, 98.8)
- added U20: ISO7320FC, Package_SO:SOIC-8_3.9x4.9mm_P1.27mm, F.Cu at (221.2, 114.9)
- added U21: IXDN614, Package_SO:SOIC-8_3.9x4.9mm_P1.27mm, F.Cu at (230.5, 122.2)
- added U22: TLV74325, Package_TO_SOT_SMD:SOT-23-5, F.Cu at (230.1, 106.6)
- added U23: LM555xM, Package_SO:SOIC-8_3.9x4.9mm_P1.27mm, F.Cu at (177.8, 145.2)
- added U24: LM555xM, Package_SO:SOIC-8_3.9x4.9mm_P1.27mm, F.Cu at (212.0, 144.1)
- added U25: LM555xM, Package_SO:SOIC-8_3.9x4.9mm_P1.27mm, F.Cu at (222.4, 144.7)
- added U26: LM555xM, Package_SO:SOIC-8_3.9x4.9mm_P1.27mm, F.Cu at (232.9, 144.9)
- added U27: LM555xM, Package_SO:SOIC-8_3.9x4.9mm_P1.27mm, F.Cu at (243.3, 144.9)
- added U28: MAX3485, Package_SO:SOIC-8_3.9x4.9mm_P1.27mm, F.Cu at (144.9, 102.1)
- added U29: MAX3485, Package_SO:SOIC-8_3.9x4.9mm_P1.27mm, F.Cu at (187.8, 80.1)
- added U3: IXDN614, Package_SO:SOIC-8_3.9x4.9mm_P1.27mm, F.Cu at (110.1, 102.8)
- added U30: MAX3485, Package_SO:SOIC-8_3.9x4.9mm_P1.27mm, F.Cu at (186.8, 105.8)
- added U4: ISO7320FC, Package_SO:SOIC-8_3.9x4.9mm_P1.27mm, F.Cu at (102.1, 102.7)
- added U5: TLV74325, Package_TO_SOT_SMD:SOT-23-5, B.Cu at (100.7, 101.4)
- added U6: MAX3485, Package_SO:SOIC-8_3.9x4.9mm_P1.27mm, F.Cu at (118.7, 102.7)
- added U8: MAX3485, Package_SO:SOIC-8_3.9x4.9mm_P1.27mm, F.Cu at (212.9, 82.3)
- J10: value Conn_02x06_Top_Bottom -> CTRL
- J11: footprint Connector_PinHeader_2.54mm:PinHeader_2x06_P2.54mm_Vertical -> Connector_PinHeader_2.54mm:PinHeader_2x06_P2.54mm_Horizontal
- J12: value Conn_01x04 -> LVIN
- J16: value Conn_01x06 -> PWMIN; footprint Connector_PinHeader_2.54mm:PinHeader_1x06_P2.54mm_Vertical -> Connector_PinHeader_2.54mm:PinHeader_1x06_P2.54mm_Horizontal
- J17: value Conn_01x06 -> HBRIDGE
- J5: value Screw_Terminal_01x02 -> BATTERY
- J6: value Screw_Terminal_01x02 -> SECONDARY
- J7: value Screw_Terminal_01x02 -> 3.3V
- Q1: value C3M0120100K -> IXFN80N50
- Q2, Q3, Q4, Q5: footprint Package_TO_SOT_THT:TO-220-3_Vertical -> Package_TO_SOT_THT:TO-220-3_Horizontal_TabDown
- R1, R2, R3: footprint Resistor_SMD:R_0603_1608Metric -> Resistor_SMD:R_2512_6332Metric
- R5: value 1.99M -> 100K; footprint Resistor_SMD:R_0603_1608Metric -> Resistor_SMD:R_2512_6332Metric
- moved J7 92.8 mm to (162.6, 155.7), turned to 0 degrees
- moved R5 78.4 mm to (115.6, 155.6), turned to 180 degrees
- moved R3 75.1 mm to (115.0, 149.5), turned to 180 degrees
- moved R1 74.2 mm to (115.1, 143.3), turned to 180 degrees
- moved J11 72.4 mm to (187.5, 145.7), turned to 90 degrees
- moved R2 67.5 mm to (114.9, 137.6), turned to 180 degrees
- moved C20 53.8 mm to (63.1, 21.9)
- moved C21 53.8 mm to (63.1, 24.4)
- moved C23 53.8 mm to (63.1, 29.4)
- moved C24 53.8 mm to (63.1, 31.9)
- moved C22 53.8 mm to (63.1, 26.9)
- moved C25 53.8 mm to (63.1, 34.4)
- moved J6 49.6 mm to (252.9, 122.6)
- moved J10 47.0 mm to (170.4, 114.4)
- moved U7 32.6 mm to (52.5, 102.9)
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Connections:
- Q1 pad 1: unconnected-(Q1-D-Pad1) -> Net-(Q1-D)
- Q1 pad 2: unconnected-(Q1-S-Pad2) -> Net-(Q1-S)
- Q1 pad 3: unconnected-(Q1-DS-Pad3) -> Net-(PS2--Vout)
- Q1 pad 4: unconnected-(Q1-G-Pad4) -> Net-(Q1-G)
- R1 pad 1: /vdc+ -> unconnected-(R1-Pad1)
- R1 pad 2: Net-(U1-INP) -> unconnected-(R1-Pad2)
- R2 pad 1: /vdc- -> unconnected-(R2-Pad1)
- R2 pad 2: /HGNDLV -> unconnected-(R2-Pad2)
- R3 pad 1: /vac+ -> unconnected-(R3-Pad1)
- R3 pad 2: Net-(U2-INP) -> unconnected-(R3-Pad2)
- R5 pad 1: /vac- -> unconnected-(R5-Pad1)
- R5 pad 2: /HGNDCV -> unconnected-(R5-Pad2)
- U12 pad 3: Net-(U12-EN) -> +3.3V
Other:
- board size 123.1 x 59.4 mm -> 182.9 x 100.4 mm
- board text added: "+"
- board text added: "-"
