File: pcb/GPC_dev_board.kicad_sch (KiCad schematic)
At the start: 83 parts, among them J1 Conn_01x12, J10 Conn_02x06_Top_Bottom, J11 Conn_02x06_Top_Bottom, J12 Conn_01x04, J13 Conn_01x04, J16 Conn_01x06, J17 Conn_01x06, J2 Conn_01x12, J3 Conn_02x13_Odd_Even, J4 Conn_02x13_Odd_Even, J5 Screw_Terminal_01x02, J6 Screw_Terminal_01x02, J7 Screw_Terminal_01x02, J8 Screw_Terminal_01x02, J9 Screw_Terminal_01x02, Q1 C3M0120100K, Q2 IRF4905, Q3 IRF4905, Q4 IRF4905, Q5 IRF4905, U1 AMC3330, U12 TLV74318, U19 XS-GPC-01, U2 AMC3330, U7 TLV74325, U9 AD7352

Commit message: In process, Dev board topology PCB sections and floorplanning evolution.
Parts:
- removed C63, C64: 10u, Capacitor_SMD:C_1206_3216Metric, symbol Device:C_Small
- removed C67, C68: 0.1u, Capacitor_SMD:C_0603_1608Metric, symbol Device:C_Small
- removed J13: Conn_01x04, Connector_PinHeader_2.54mm:PinHeader_1x04_P2.54mm_Vertical, symbol Connector_Generic:Conn_01x04
- removed J8, J9: Screw_Terminal_01x02, TerminalBlock_Phoenix:TerminalBlock_Phoenix_MKDS-1,5-2-5.08_1x02_P5.08mm_Horizontal, symbol Connector:Screw_Terminal_01x02
- removed R43: 10K, Resistor_SMD:R_0603_1608Metric, symbol Device:R
- added C26, C27, C29, C37, C9: C_Polarized, Capacitor_THT:CP_Radial_D10.0mm_P5.00mm, symbol Device:C_Polarized
- added C3, C34, C35, C40, C41, C42, C45, C46, C47, C50, C51, C54, C55: 0.1u, Capacitor_SMD:C_0603_1608Metric, symbol Device:C_Small
- added C30: 22n 1000v, Capacitor_THT:C_Rect_L13.0mm_W6.0mm_P10.00mm_FKS3_FKP3_MKS4, symbol Device:C_Polarized_Small
- added C31, C38, C43, C48: 1u, Capacitor_SMD:C_0603_1608Metric, symbol Device:C_Small
- added C33, C39, C44, C49: 0.01u, Capacitor_SMD:C_0603_1608Metric, symbol Device:C_Small
- added C58, C60, C62: 2.2n 80V, Capacitor_SMD:C_0603_1608Metric, symbol Device:C_Small
- added D1: DC UNDER, LED_SMD:LED_0603_1608Metric, symbol Device:LED
- added D2: DC OVER, LED_SMD:LED_0603_1608Metric, symbol Device:LED
- added D3: AC UNDER, LED_SMD:LED_0603_1608Metric, symbol Device:LED
- added D4: AC OVER, LED_SMD:LED_0603_1608Metric, symbol Device:LED
- added D5: 3.3V, LED_SMD:LED_0603_1608Metric, symbol Device:LED
- added H1, H10, H11, H13, H14, H15, H16, H2, H3, H4, H5, H6, H7, H9: ~, MountingHole:MountingHole_3mm_Pad, symbol Mechanical:MountingHole_Pad
- added J14: Conn_01x04, Connector_PinHeader_2.54mm:PinHeader_1x04_P2.54mm_Horizontal, symbol Connector_Generic:Conn_01x04
- added J15: Vdc, TerminalBlock_Phoenix:TerminalBlock_Phoenix_MKDS-1,5-2-5.08_1x02_P5.08mm_Horizontal, symbol Connector:Screw_Terminal_01x02
- added J18: Vac, TerminalBlock_Phoenix:TerminalBlock_Phoenix_MKDS-1,5-2-5.08_1x02_P5.08mm_Horizontal, symbol Connector:Screw_Terminal_01x02
- added J19: LVIN, Connector_PinHeader_2.54mm:PinHeader_1x04_P2.54mm_Vertical, symbol Connector_Generic:Conn_01x04
- added J20: LVOUT, Connector_PinHeader_2.54mm:PinHeader_1x04_P2.54mm_Horizontal, symbol Connector_Generic:Conn_01x04
- added PS1, PS2, PS3, PS4: RM-3.312S, Converter_DCDC:Converter_DCDC_Murata_MEE1SxxxxSC_THT, symbol Converter_DCDC:MEE1S1212SC
- added Q6, Q7, Q8, Q9: MMBT3904, Package_TO_SOT_SMD:SOT-23, symbol Transistor_BJT:MMBT3904
- added R10, R11, R17, R18, R21, R22: 47K, Resistor_SMD:R_0603_1608Metric, symbol Device:R
- added R15, R19, R23, R27, R28: 100R, Resistor_SMD:R_0603_1608Metric, symbol Device:R
- added R16, R20, R24, R25, R26: 10R, Resistor_SMD:R_0603_1608Metric, symbol Device:R
- added R4: 1.99M, Resistor_SMD:R_2512_6332Metric, symbol Device:R
- added R6: 100K, Resistor_SMD:R_2512_6332Metric, symbol Device:R
- added R9: 150R 3W, Resistor_SMD:R_2512_6332Metric, symbol Device:R_US
- added RV1: GAIN_SIN, Potentiometer_THT:Potentiometer_Bourns_3299X_Horizontal, symbol Device:R_Potentiometer_US
- added RV2: GAIN_OUT, Potentiometer_THT:Potentiometer_Bourns_3299X_Horizontal, symbol Device:R_Potentiometer_US
- added RV3: GAIN_AC, Potentiometer_THT:Potentiometer_Bourns_3299X_Horizontal, symbol Device:R_Potentiometer_US
- added RV4: GAIN_DC, Potentiometer_THT:Potentiometer_Bourns_3299X_Horizontal, symbol Device:R_Potentiometer_US
- added RV5: PWM_VREF, Potentiometer_THT:Potentiometer_Bourns_3299X_Horizontal, symbol Device:R_Potentiometer_US
- added U10, U15, U20, U4: ISO7320FC, Package_SO:SOIC-8_3.9x4.9mm_P1.27mm, symbol Isolator:ISO7320FC
- added U11, U16, U22, U5: TLV74325, Package_TO_SOT_SMD:SOT-23-5, symbol myspace:TLV74325_SOT23-5
- added U13, U17, U18, U21, U3: IXDN614, Package_SO:SOIC-8_3.9x4.9mm_P1.27mm, symbol myspace:IR2125
- added U14, U28, U29, U30, U6, U8: MAX3485, Package_SO:SOIC-8_3.9x4.9mm_P1.27mm, symbol Interface_UART:MAX3485
- added U23, U24, U25, U26, U27: LM555xM, Package_SO:SOIC-8_3.9x4.9mm_P1.27mm, symbol Timer:LM555xM
- J10: value Conn_02x06_Top_Bottom -> CTRL
- J11: footprint Connector_PinHeader_2.54mm:PinHeader_2x06_P2.54mm_Vertical -> Connector_PinHeader_2.54mm:PinHeader_2x06_P2.54mm_Horizontal
- J12: value Conn_01x04 -> LVIN
- J16: value Conn_01x06 -> PWMIN; footprint Connector_PinHeader_2.54mm:PinHeader_1x06_P2.54mm_Vertical -> Connector_PinHeader_2.54mm:PinHeader_1x06_P2.54mm_Horizontal
- J17: value Conn_01x06 -> HBRIDGE
- J5: value Screw_Terminal_01x02 -> BATTERY
- J6: value Screw_Terminal_01x02 -> SECONDARY
- J7: value Screw_Terminal_01x02 -> 3.3V
- Q1: value C3M0120100K -> IXFN80N50
- Q2, Q3, Q4, Q5: footprint Package_TO_SOT_THT:TO-220-3_Vertical -> Package_TO_SOT_THT:TO-220-3_Horizontal_TabDown
- R1, R2, R3: footprint Resistor_SMD:R_0603_1608Metric -> Resistor_SMD:R_2512_6332Metric
- R5: value 1.99M -> 100K; footprint Resistor_SMD:R_0603_1608Metric -> Resistor_SMD:R_2512_6332Metric
Connections:
- net +3.3V: now also U12.3 (EN), J14.1 (Pin_1), R10.2, R11.2, R21.2
- net GND: now also C31.2, C33.2, C34.2, C38.2, C39.2, C43.2, C44.2, C48.2, C49.2, J14.4 (Pin_4), PS1.1 (-Vin), PS2.1 (-Vin), PS3.1 (-Vin), PS4.1 (-Vin), R17.1, R18.1, R22.1, U5.2 (GND), U8.2 (~{RE}), U8.3 (DE), U8.4 (DI)
- net HGNDCV: no longer R5.2
- net HGNDLV: no longer R2.2
- net pwm: now also U4.7 (OUTA)
- net vac+: no longer R3.1
- net vac-: no longer R5.1
- net vdc+: no longer R1.1
- net vdc-: no longer R2.1
- net at R7.2, U1.6 (INP): no longer R1.2
- net at R8.2, U2.6 (INP): no longer R3.2
- net at Q1.1 (D): now also C30.1
- net at Q1.2 (S): now also R9.2
- net at Q1.3 (DS): now also C35.2, PS2.3 (-Vout)
- net at Q1.4 (G): now also R16.2
- new net: C38.1, C39.1, PS1.2 (+Vin)
- new net: C43.1, C44.1, PS3.2 (+Vin)
- new net: C47.2, PS3.3 (-Vout)
- new net: C47.1, PS3.4 (+Vout)
- new net: U10.2 (INA), U8.1 (RO)
- new net: R22.2, R23.1, U14.6 (A)
- new net: R21.1, R23.2, U14.7 (B)
- new net: C42.2, PS1.3 (-Vout)
- new net: C42.1, PS1.4 (+Vout)
- new net: C48.1, C49.1, PS4.2 (+Vin)
- new net: C31.1, C33.1, PS2.2 (+Vin)
- new net: R18.2, R19.1, U8.6 (A)
- new net: R10.1, R19.2, U8.7 (B)
- new net: U4.2 (INA), U6.1 (RO)
- new net: R15.1, R17.2, U6.6 (A)
- new net: J14.2 (Pin_2), R11.1, R15.2, U6.7 (B)
- new net: C35.1, PS2.4 (+Vout)
- new net: C30.2, R9.1
- new net: C54.1, PS4.4 (+Vout)
- new net: C54.2, PS4.3 (-Vout)
- no-connect marks 15 -> 34
Other:
- note added: "Connector 0.6" DIP-24"
- note added: "Control Interface"
- note added: "Dump FET"
- note added: "Emmulator Connector"
- note added: "GPC-XB Board"
- note added: "Hbridge"
- note added: "Hbridge Driver"
- note added: "Voltage Dividers"
- note removed: "Emulator Connector"
- note removed: "Experiment Board Connector 0.6" DIP-24"
- moved on the sheet: C14, C16, C22, C24, C28, C32, C36, C4, C5, C52, C53, C56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
